Commit message: Working Ackermann vehicle, controllers and all.

File: ack_description/urdf/gem.xacro (robot description, xacro)
@@ -41,33 +41,4 @@
   <xacro:wheel name="${lr}" radius="${wheel_diameter/2}" width="${wheel_thickness}" material="Gazebo/Blue" />
   <xacro:wheel name="${lr}_assembly" radius="0.1" width="0.001" material="Gazebo/White" />
-	<!--<link name="${lr}_assembly">
-		<collision>
-		  <origin xyz="0 0 0" rpy="0 1.5708 1.5708" />
-		  <geometry>
-		   <cylinder length="0.001" radius="0.1"/>
-		  </geometry>
-		</collision>
-		<visual>
-		  <origin xyz="0 0 0" rpy="0 1.5708 1.5708" />
-		  <geometry>
-			<cylinder length="0.001" radius="0.1"/>
-		  </geometry>
-		  <material name="white"/>
-		</visual>
-		<inertial>
-		  <origin xyz="0 0 0" rpy="0 1.5708 1.5708" />
-		  <mass value="0.2"/>
-		  <cylinder_inertia m="0.2" r="0.3" h="0.1"/>
-      <inertia ixx="0.4" ixy="0.1" ixz="0.1" iyy="0.4" iyz="0.1" izz="0.2"/>
-	  </inertial>
-	</link>
-  <gazebo reference="${lr}_assembly">
-    <mu1 value="2.0"/>
-    <mu2 value="2.0"/>
-    <kp  value="10000000.0" />
-    <kd  value="1.0" />
-    <fdir1 value="0 1 0"/>
-    <material>Gazebo/White</material>
-  </gazebo>-->
   <joint name="${lr}_hinge" type="revolute">
     <parent link="chassis"/>
@@ -88,5 +59,5 @@
   <transmission name="trans_${lr}_hing">
     <type>transmission_interface/SimpleTransmission</type>
-    <joint name="right_wheel_hinge">
+    <joint name="${lr}_hinge">
       <hardwareInterface>EffortJointInterface</hardwareInterface>
     </joint>
@@ -98,5 +69,5 @@
   <transmission name="trans_${lr}_rotate">
     <type>transmission_interface/SimpleTransmission</type>
-    <joint name="${lr}">
+    <joint name="${lr}_rotate">
       <hardwareInterface>EffortJointInterface</hardwareInterface>
     </joint>
@@ -106,4 +77,15 @@
     </actuator>
   </transmission>
+</xacro:macro>
+<xacro:macro name="rear_wheel" params="lr lr_reflect">
+  <xacro:wheel name="${lr}" radius="${wheel_diameter/2}" width="${wheel_thickness}" material="Gazebo/Blue" />
+  <joint name="${lr}_rotate" type="continuous">
+    <parent link="chassis"/>
+    <child link="${lr}"/>
+    <origin xyz="${-wheel_base_length/2} ${lr_reflect*((wheel_base_width/2)+(wheel_thickness/2))} ${wheel_diameter/2}" rpy="0 0 0" />
+    <axis xyz="0 1 0" rpy="0 0 0" />
+    <limit effort="0" velocity="0"/>
+    <dynamics damping="0.0" friction="0.0"/>
+  </joint>
 </xacro:macro>
 <!-- Macros End -->
@@ -156,3 +138,12 @@
 	<!-- Chassis END -->
   <xacro:wheel_steer lr="right_wheel" lr_reflect="-1" />
+  <xacro:wheel_steer lr="left_wheel" lr_reflect="1" />
+  <xacro:rear_wheel lr="right_wheel_rear" lr_reflect="-1" />
+  <xacro:rear_wheel lr="left_wheel_rear" lr_reflect="1" />
+  <gazebo>
+		<plugin name="gazebo_ros_control" filename="libgazebo_ros_control.so">
+		  <robotNamespace>/ack</robotNamespace>
+			<legacyModeNS>true</legacyModeNS>
+		</plugin>
+	</gazebo>
 </robot>
