Commit message: Adjustments...

File: ack_description/urdf/gem_1kg_LiDAR.xacro (robot description, xacro)
@@ -64,5 +64,5 @@
     </joint>
     <actuator name="motor_${lr}_front">
-      <hardwareInterface>hardware_interface/EffortJointInterface</hardwareInterface>
+      <!--<hardwareInterface>hardware_interface/EffortJointInterface</hardwareInterface>-->
       <mechanicalReduction>1</mechanicalReduction>
     </actuator>
@@ -74,5 +74,5 @@
     </joint>
     <actuator name="motor_${lr}_rotate">
-      <hardwareInterface>hardware_interface/EffortJointInterface</hardwareInterface>
+      <!--<hardwareInterface>hardware_interface/EffortJointInterface</hardwareInterface>-->
       <mechanicalReduction>1</mechanicalReduction>
     </actuator>
@@ -152,5 +152,5 @@
     <dampingFactor>0</dampingFactor>
     <material>Gazebo/White</material>
-    <selfCollide>true</selfCollide>
+    <selfCollide>false</selfCollide>
     <turnGravityOff>false</turnGravityOff>
     <mu1 value="0.1"/>
@@ -163,10 +163,4 @@
   <xacro:rear_wheel lr="right_wheel_rear" lr_reflect="-1" />
   <xacro:rear_wheel lr="left_wheel_rear" lr_reflect="1" />
-  <gazebo>
-		<plugin name="gazebo_ros_control" filename="libgazebo_ros_control.so">
-		  <robotNamespace>/ack</robotNamespace>
-			<legacyModeNS>true</legacyModeNS>
-		</plugin>
-	</gazebo>
   	<!-- Camera -->
 	<!-- You can adjust the camera angle with the p in rpy, measured in radians. -->
@@ -258,4 +252,19 @@
                izz="1.0" />
     </inertial>
-  </link>
+  </link><!---->
+    <gazebo>
+		<plugin name="gazebo_ros_control" filename="libgazebo_ros_control.so">
+		  <robotNamespace>/ack</robotNamespace>
+			<legacyModeNS>true</legacyModeNS>
+		</plugin>
+	</gazebo>
+  <!--<gazebo>
+    <plugin filename="libgazebo_ros_control.so" name="ros_control">
+      <robotNamespace>/ack</robotNamespace>
+      <robotParam>/ack/gem</robotParam>
+      <controlPeriod>0.001</controlPeriod>
+      <robotSimType>gazebo_ros_control/DefaultRobotHWSim</robotSimType>
+      <legacyModeNS>true</legacyModeNS>
+    </plugin>
+  </gazebo>-->
 </robot>
